Commit message: Added tags for the gazebo in the xacro

File: description/robot_core.xacro (robot description, xacro)
@@ -41,4 +41,7 @@
         <axis xyz="0.0 0.0 0.0"/>
     </joint>
+    <gazebo reference="chassis">
+        <material>Gazebo/White</material>
+    </gazebo>
     <!-- Left Wheel Link -->
     <joint name="left_wheel_joint" type="continuous">
@@ -65,4 +68,7 @@
         </xacro:inertial_cylinder>
     </link>
+    <gazebo reference="left_wheel">
+        <material>Gazebo/Blue</material>
+    </gazebo>
     <!-- Right Wheel Link -->
     <joint name="right_wheel_joint" type="continuous">
@@ -89,4 +95,7 @@
         </xacro:inertial_cylinder>
     </link>
+    <gazebo reference="right_wheel">
+        <material>Gazebo/Blue</material>
+    </gazebo>
     <!-- Castor Wheel Link -->
     <joint name="castor_wheel_joint" type="fixed">
@@ -111,3 +120,6 @@
         </xacro:inertial_sphere>
     </link>
+    <gazebo reference="castor_wheel">
+        <material>Gazebo/Black</material>
+    </gazebo>
 </robot>

Commit message: Corrected wheel slippage

File: description/robot_core.xacro (robot description, xacro)
@@ -64,5 +64,5 @@
             <origin xyz="0.0 0.0 0.0" rpy="0.0 0.0 0.0"/>
             <geometry>
-                <cylinder radius="0.05" length="0.04"/>
+                <sphere radius="0.05"/>
             </geometry>
         </collision>
@@ -91,5 +91,5 @@
             <origin xyz="0.0 0.0 0.0" rpy="0.0 0.0 0.0"/>
             <geometry>
-                <cylinder radius="0.05" length="0.04"/>
+                <sphere radius="0.05"/>
             </geometry>
         </collision>

Commit message: Using SLAM for localization and mapping

File: description/robot_core.xacro (robot description, xacro)
@@ -19,4 +19,11 @@
     <!-- Base Link -->
     <link name="base_link"/>
+    <!-- Base Footprint -->
+    <joint name="base_footprint_joint" type="fixed">
+        <origin xyz="0.0 0.0 0.0" rpy="0.0 0.0 0.0"/>
+        <parent link="base_link"/>
+        <child link="base_footprint"/>
+    </joint>
+    <link name="base_footprint"/>
     <!-- Chassis Link -->
     <link name="chassis">
